File: PLACA_IEMA.kicad_sch (KiCad schematic)
At the start: 7 parts, among them J1 Conn_02x14_Odd_Even, U1 esp32-wemos-d1-mini, U2 module_bme280, U3 module_mpu6050, U4 HMC5883L, U5 YAAJ_DCDC_StepDown_LM2596

Commit message: alterações dia 22/10/2026
Connections:
- net RX_RS485 is gone; now on net SPI/MOSI: U1.28 (IO_32)
- net I2C_SCL_1: now also J1.24 (Pin_24)
- net I2C_SDA_1: now also U1.26 (IO_25)
- net SPI/MOSI: now also J1.23 (Pin_23)
- net RS485_RX: no longer names the net of J1.8 (Pin_8)
- net RS485_TX: no longer names the net of J1.7 (Pin_7)
- no-connect marks 49 -> 48
Changed lines of the file:
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@@
+	)
+	(no_connect
+		(at 154.94 81.28)
 	)
 	(no_connect
@@
 	)
 	(no_connect
-		(at 167.64 101.6)
-	)
-	(no_connect
 		(at 167.64 88.9)
 	)
@@
 	)
 	(no_connect
-		(at 106.68 111.76)
-	)
-	(no_connect
 		(at 189.23 120.65)
 	)
@@
 	)
 	(no_connect
+		(at 167.64 81.28)
+	)
+	(no_connect
 		(at 133.35 72.39)
 	)
@@
 	(no_connect
 		(at 154.94 76.2)
-	)
-	(no_connect
-		(at 154.94 101.6)
 	)
 	(no_connect
@@
 		)
 	)
-	(label "RS485_RX"
-		(at 167.64 81.28 0)
-		(effects
-			(font
-				(size 1.27 1.27)
-			)
-			(justify left bottom)
-		)
-	)
 	(label "I2C_SDA_1"
 		(at 189.23 113.03 180)
@@
 		)
 	)
+	(label "I2C_SDA_1"
+		(at 106.68 111.76 180)
+		(effects
+			(font
+				(size 1.27 1.27)
+			)
+			(justify right bottom)
+		)
+	)
 	(label "GND"
 		(at 133.35 66.04 0)
@@
 			)
 			(justify left bottom)
+		)
+	)
+	(label "SPI{slash}MOSI"
+		(at 154.94 101.6 180)
+		(effects
+			(font
+				(size 1.27 1.27)
+			)
+			(justify right bottom)
 		)
 	)
@@
 		)
 	)
-	(label "RS485_TX"
-		(at 154.94 81.28 180)
-		(effects
-			(font
-				(size 1.27 1.27)
-			)
-			(justify right bottom)
+	(label "I2C_SCL_1"
+		(at 167.64 101.6 0)
+		(effects
+			(font
+				(size 1.27 1.27)
+			)
+			(justify left bottom)
 		)
 	)
@@
 		)
 	)
-	(label "RX_RS485"
+	(label "SPI{slash}MOSI"
 		(at 106.68 88.9 180)
 		(effects

Commit message: Alterações de Pino
Connections:
- net I2C_SCL_1: now also J1.27 (Pin_27); no longer J1.24 (Pin_24)
- net I2C_SDA_1: now also J1.28 (Pin_28)
- net SPI/MOSI: no longer J1.23 (Pin_23)
- no-connect marks 48 -> 50
Changed lines of the file:
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@@
+	)
+	(no_connect
+		(at 154.94 101.6)
 	)
 	(no_connect
@@
 	(no_connect
 		(at 133.35 74.93)
+	)
+	(no_connect
+		(at 167.64 101.6)
 	)
 	(no_connect
@@
 		)
 	)
+	(label "I2C_SDA_1"
+		(at 167.64 106.68 0)
+		(effects
+			(font
+				(size 1.27 1.27)
+			)
+			(justify left bottom)
+		)
+	)
 	(label "TX_RS485"
 		(at 106.68 81.28 180)
@@
 		)
 	)
+	(label "I2C_SCL_1"
+		(at 154.94 106.68 180)
+		(effects
+			(font
+				(size 1.27 1.27)
+			)
+			(justify right bottom)
+		)
+	)
 	(label "I2C_SDA_1"
 		(at 106.68 104.14 180)
@@
 		)
 	)
-	(label "SPI{slash}MOSI"
-		(at 154.94 101.6 180)
-		(effects
-			(font
-				(size 1.27 1.27)
-			)
-			(justify right bottom)
-		)
-	)
 	(label "GND"
 		(at 133.35 60.96 0)
@@
 		(effects
 			(font
-				(size 1.27 1.27)
-			)
-			(justify left bottom)
-		)
-	)
-	(label "I2C_SCL_1"
-		(at 167.64 101.6 0)
-		(effects
-			(font
